File: Hardware/SparkFun_ProtoShield_Kit_rev40.sch (EAGLE design)
At the start: 105 parts, among them SW2 MOMENTARY-SWITCH-SPST-PTH-6.0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

Commit message: Update to v40
-Update SCH version number
-Update BRD version number in copper
-Update file names
Other:
- note added: "v40"
- note removed: "v32"
Changed lines of the file:
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@@
 <?xml version="1.0" encoding="utf-8"?>
 <!DOCTYPE eagle SYSTEM "eagle.dtd">
-<eagle version="7.7.0">
+<eagle version="7.6.0">
 <drawing>
 <settings>
@@
 <setting verticaltext="up"/>
 </settings>
-<grid distance="0.01" unitdist="inch" unit="inch" style="lines" multiple="1" display="no" altdistance="0.01" altunitdist="inch" altunit="inch"/>
+<grid distance="0.1" unitdist="inch" unit="inch" style="lines" multiple="1" display="no" altdistance="0.01" altunitdist="inch" altunit="inch"/>
 <layers>
 <layer number="1" name="Top" color="4" fill="1" visible="no" active="no"/>
@@
 <plain>
 <text x="170.942" y="11.43" size="2.54" layer="94" font="vector">Nathan Seidle</text>
-<text x="238.76" y="7.62" size="2.54" layer="94" font="vector">v32</text>
+<text x="238.76" y="7.62" size="2.54" layer="94" font="vector">v40</text>
 <text x="170.688" y="7.62" size="1.778" layer="94" font="vector" ratio="7">Toni Klopfenstein &amp; Ho Yun "Bobby" Chan</text>
 <text x="38.1" y="170.18" size="2.032" layer="97" font="vector" ratio="15">Arduino Shield</text>
